Commit message: Added a lot

File: henry/urdf/camera.xacro (robot description, xacro)
@@ -6,5 +6,5 @@
       <origin xyz="0 0 0" rpy="0 0 0"/>
       <geometry>
-    <box size="0.025 0.075 0.025"/>
+        <box size="0.025 0.075 0.025"/>
       </geometry>
     </collision>
@@ -43,5 +43,5 @@
         <frameName>camera_link</frameName>
         <pointCloudCutoff>0.5</pointCloudCutoff>
-        <pointCloudCutoffMax>3.0</pointCloudCutoffMax>
+        <pointCloudCutoffMax>20.0</pointCloudCutoffMax>
         <distortionK1>0</distortionK1>
         <distortionK2>0</distortionK2>
@@ -55,15 +55,15 @@
         <hackBaseline>0</hackBaseline>
       </plugin>
-      <update_rate>20</update_rate>
+      <update_rate>10</update_rate>
       <camera>
-        <horizontal_fov>1.047198</horizontal_fov>
+        <horizontal_fov>1.57079632679</horizontal_fov>
         <image>
-          <width>640</width>
-          <height>480</height>
+          <width>100</width>
+          <height>80</height>
           <format>R8G8B8</format>
         </image>
         <clip>
           <near>0.05</near>
-          <far>3</far>
+          <far>20</far>
         </clip>
       </camera>

File: henry/urdf/henry.xacro (robot description, xacro)
@@ -5,4 +5,7 @@
 <robot name="henry" xmlns:xacro="http://www.ros.org/wiki/xacro">
   <xacro:property name="inertMult" value="2"/>
+  <xacro:property name="j1Effort" value="4"/>
+  <xacro:property name="j2Effort" value="6"/>
+  <xacro:property name="j3Effort" value="4"/>
   <xacro:include filename="$(find henry)/urdf/macros.xacro" />
   <xacro:include filename="$(find henry)/urdf/camera.xacro" />
@@ -112,5 +115,5 @@
       lower="-1.719147861"
       upper="1.719147861"
-      effort="2"
+      effort="${j1Effort}"
       velocity="0"/>
   </joint>
@@ -169,5 +172,5 @@
       lower="-1.719147861"
       upper="1.719147861"
-      effort="2"
+      effort="${j2Effort}"
       velocity="0"/>
   </joint>
@@ -222,9 +225,9 @@
       link="rf3" />
     <axis
-      xyz="0 0 1" />
-    <limit
-      lower="-1.719147861"
-      upper="1.719147861"
-      effort="2"
+      xyz="0 0 -1" />
+    <limit
+      lower="-1.719147861"
+      upper="1.719147861"
+      effort="${j3Effort}"
       velocity="0"/>
   </joint>
@@ -283,5 +286,5 @@
       lower="-1.719147861"
       upper="1.719147861"
-      effort="2"
+      effort="${j1Effort}"
       velocity="0"/>
   </joint>
@@ -340,5 +343,5 @@
       lower="-1.719147861"
       upper="1.719147861"
-      effort="2"
+      effort="${j2Effort}"
       velocity="0"/>
   </joint>
@@ -393,9 +396,9 @@
       link="rc3" />
     <axis
-      xyz="0 0 1" />
-    <limit
-      lower="-1.719147861"
-      upper="1.719147861"
-      effort="2"
+      xyz="0 0 -1" />
+    <limit
+      lower="-1.719147861"
+      upper="1.719147861"
+      effort="${j3Effort}"
       velocity="0"/>
   </joint>
@@ -454,5 +457,5 @@
       lower="-1.719147861"
       upper="1.719147861"
-      effort="2"
+      effort="${j1Effort}"
       velocity="0"/>
   </joint>
@@ -511,5 +514,5 @@
       lower="-1.719147861"
       upper="1.719147861"
-      effort="2"
+      effort="${j2Effort}"
       velocity="0"/>
   </joint>
@@ -564,9 +567,9 @@
       link="rr3" />
     <axis
-      xyz="0 0 1" />
-    <limit
-      lower="-1.719147861"
-      upper="1.719147861"
-      effort="2"
+      xyz="0 0 -1" />
+    <limit
+      lower="-1.719147861"
+      upper="1.719147861"
+      effort="${j3Effort}"
       velocity="0"/>
   </joint>
@@ -625,5 +628,5 @@
       lower="-1.719147861"
       upper="1.719147861"
-      effort="2"
+      effort="${j1Effort}"
       velocity="0"/>
   </joint>
@@ -682,5 +685,5 @@
       lower="-1.719147861"
       upper="1.719147861"
-      effort="2"
+      effort="${j2Effort}"
       velocity="0"/>
   </joint>
@@ -735,9 +738,9 @@
       link="lf3" />
     <axis
-      xyz="0 0 1" />
-    <limit
-      lower="-1.719147861"
-      upper="1.719147861"
-      effort="2"
+      xyz="0 0 -1" />
+    <limit
+      lower="-1.719147861"
+      upper="1.719147861"
+      effort="${j3Effort}"
       velocity="0"/>
   </joint>
@@ -796,5 +799,5 @@
       lower="-1.719147861"
       upper="1.719147861"
-      effort="2"
+      effort="${j1Effort}"
       velocity="0"/>
   </joint>
@@ -853,5 +856,5 @@
       lower="-1.719147861"
       upper="1.719147861"
-      effort="2"
+      effort="${j2Effort}"
       velocity="0"/>
   </joint>
@@ -906,9 +909,9 @@
       link="lc3" />
     <axis
-      xyz="0 0 1" />
-    <limit
-      lower="-1.719147861"
-      upper="1.719147861"
-      effort="2"
+      xyz="0 0 -1" />
+    <limit
+      lower="-1.719147861"
+      upper="1.719147861"
+      effort="${j3Effort}"
       velocity="0"/>
   </joint>
@@ -967,5 +970,5 @@
       lower="-1.719147861"
       upper="1.719147861"
-      effort="2"
+      effort="${j1Effort}"
       velocity="0"/>
   </joint>
@@ -1024,5 +1027,5 @@
       lower="-1.719147861"
       upper="1.719147861"
-      effort="2"
+      effort="${j2Effort}"
       velocity="0"/>
   </joint>
@@ -1077,9 +1080,9 @@
       link="lr3" />
     <axis
-      xyz="0 0 1" />
-    <limit
-      lower="-1.719147861"
-      upper="1.719147861"
-      effort="2"
+      xyz="0 0 -1" />
+    <limit
+      lower="-1.719147861"
+      upper="1.719147861"
+      effort="${j3Effort}"
       velocity="0"/>
   </joint>
@@ -1087,30 +1090,30 @@
     <mu1>999999</mu1>
     <mu2>999999</mu2>
-    <minDepth>0.01</minDepth>
+    <minDepth>0.02</minDepth>
   </gazebo>
   <gazebo reference="rc3">
     <mu1>999999</mu1>
     <mu2>999999</mu2>
-    <minDepth>0.01</minDepth>
+    <minDepth>0.02</minDepth>
   </gazebo>
   <gazebo reference="rr3">
     <mu1>999999</mu1>
     <mu2>999999</mu2>
-    <minDepth>0.01</minDepth>
+    <minDepth>0.02</minDepth>
   </gazebo>
   <gazebo reference="lf3">
     <mu1>999999</mu1>
     <mu2>999999</mu2>
-    <minDepth>0.01</minDepth>
+    <minDepth>0.02</minDepth>
   </gazebo>
   <gazebo reference="lc3">
     <mu1>999999</mu1>
     <mu2>999999</mu2>
-    <minDepth>0.01</minDepth>
+    <minDepth>0.02</minDepth>
   </gazebo>
   <gazebo reference="lr3">
     <mu1>999999</mu1>
     <mu2>999999</mu2>
-    <minDepth>0.01</minDepth>
+    <minDepth>0.02</minDepth>
   </gazebo>
   <trans name = "rf1"/>

File: henry/urdf/macros.xacro (robot description, xacro)
@@ -9,5 +9,5 @@
             <actuator name="${name}Motor">
                 <hardwareInterface>hardware_interface/EffortJointInterface</hardwareInterface>
-                <mechanicalReduction>10</mechanicalReduction>
+                <mechanicalReduction>10000</mechanicalReduction>
             </actuator>
         </transmission>

Commit message: Final

File: henry/urdf/camera.xacro (robot description, xacro)
@@ -37,11 +37,6 @@
         <updateRate>0.0</updateRate>
         <cameraName>camera_ir</cameraName>
-        <imageTopicName>/camera/color/image_raw</imageTopicName>
         <depthImageTopicName>/camera/depth/image_raw</depthImageTopicName>
-        <depthImageCameraInfoTopicName>/camera/depth/camera_info</depthImageCameraInfoTopicName>
-        <pointCloudTopicName>/camera/depth/points</pointCloudTopicName>
         <frameName>camera_link</frameName>
-        <pointCloudCutoff>0.5</pointCloudCutoff>
-        <pointCloudCutoffMax>20.0</pointCloudCutoffMax>
         <distortionK1>0</distortionK1>
         <distortionK2>0</distortionK2>

File: henry/urdf/henry.xacro (robot description, xacro)
@@ -5,7 +5,7 @@
 <robot name="henry" xmlns:xacro="http://www.ros.org/wiki/xacro">
   <xacro:property name="inertMult" value="2"/>
-  <xacro:property name="j1Effort" value="4"/>
-  <xacro:property name="j2Effort" value="6"/>
-  <xacro:property name="j3Effort" value="4"/>
+  <xacro:property name="j1Effort" value="3"/>
+  <xacro:property name="j2Effort" value="4"/>
+  <xacro:property name="j3Effort" value="2"/>
   <xacro:include filename="$(find henry)/urdf/macros.xacro" />
   <xacro:include filename="$(find henry)/urdf/camera.xacro" />
@@ -1088,31 +1088,31 @@
   </joint>
   <gazebo reference="rf3">
-    <mu1>999999</mu1>
-    <mu2>999999</mu2>
+    <mu1>9999999999999999</mu1>
+    <mu2>9999999999999999</mu2>
     <minDepth>0.02</minDepth>
   </gazebo>
   <gazebo reference="rc3">
-    <mu1>999999</mu1>
-    <mu2>999999</mu2>
+    <mu1>9999999999999999</mu1>
+    <mu2>9999999999999999</mu2>
     <minDepth>0.02</minDepth>
   </gazebo>
   <gazebo reference="rr3">
-    <mu1>999999</mu1>
-    <mu2>999999</mu2>
+    <mu1>9999999999999999</mu1>
+    <mu2>9999999999999999</mu2>
     <minDepth>0.02</minDepth>
   </gazebo>
   <gazebo reference="lf3">
-    <mu1>999999</mu1>
-    <mu2>999999</mu2>
+    <mu1>9999999999999999</mu1>
+    <mu2>9999999999999999</mu2>
     <minDepth>0.02</minDepth>
   </gazebo>
   <gazebo reference="lc3">
-    <mu1>999999</mu1>
-    <mu2>999999</mu2>
+    <mu1>9999999999999999</mu1>
+    <mu2>9999999999999999</mu2>
     <minDepth>0.02</minDepth>
   </gazebo>
   <gazebo reference="lr3">
-    <mu1>999999</mu1>
-    <mu2>999999</mu2>
+    <mu1>9999999999999999</mu1>
+    <mu2>9999999999999999</mu2>
     <minDepth>0.02</minDepth>
   </gazebo>
